Commit message: i added ros2 control

File: amr_description/urdf/amr_camera.urdf.xacro (robot description, xacro)
@@ -1,10 +1,13 @@
 <?xml version="1.0"?>
 <robot xmlns:xacro="http://www.ros.org/wiki/xacro">
+<xacro:property name="camera_length" value="0.04"/>
+<xacro:property name="camera_width" value="0.02"/>
+<xacro:property name="camera_height" value="0.035"/>
     <link name="camera_link">
         <visual>
             <geometry>
-                <box size="0.02 0.02 0.035"/>
+                <box size="${camera_length} ${camera_width} ${camera_height}"/>
             </geometry>
-            <origin xyz="0.0 0.0 0.0" rpy="0.0 0.0 0.0"/>
+            <origin xyz="0.0 0.0 0.0" rpy="0.0 0.0 ${pi/2}"/>
             <material name="black">
                 <color rgba="0.0 0.0 0.0 1.0"/>
@@ -13,13 +16,13 @@
         <collision>
             <geometry>
-                <box size="0.02 0.02 0.035"/>
+                <box size="${camera_length} ${camera_width} ${camera_height}"/>
             </geometry>
-            <origin xyz="0.0 0.0 0.0" rpy="0.0 0.0 0.0"/>
+            <origin xyz="0.0 0.0 0.0" rpy="0.0 0.0 ${pi/2}"/>
         </collision>
-        <xacro:box m="0.2" l="0.02" w="0.02" h="0.035" xyz="0.0 0.0 0.0" rpy="0.0 0.0 0.0"/>
+        <xacro:box m="0.2" l="0.02" w="0.02" h="0.035" xyz="0.0 0.0 0.0" rpy="0.0 0.0 ${pi/2}"/>
     </link>
     <joint name="base_top_camera_joint" type="fixed">
-        <origin xyz="0.25 0.0 0.0175" rpy="0.0 0.0 0.0"/>
-        <parent link="base_top_link"/>
+       <origin xyz="0.0 ${chassis_width/2} 0.0" rpy="0.0 0.0 ${pi/2}"/>
+        <parent link="chassis_top"/>
         <child link="camera_link"/>
     </joint>

File: amr_description/urdf/amr_gazebo.urdf.xacro (robot description, xacro)
@@ -1,20 +1,20 @@
 <?xml version="1.0"?>
 <robot xmlns:xacro="http://www.ros.org/wiki/xacro">
-    <gazebo reference="base_bottom_link">
+    <gazebo reference="chassis_base">
         <material>Gazebo/Silver</material>
     </gazebo>
-    <gazebo reference="base_top_link">
+    <gazebo reference="chassis_top">
         <material>Gazebo/Silver</material>
     </gazebo>
-    <gazebo reference="front_left_tire_link">
+    <gazebo reference="front_left_wheel_link">
         <material>Gazebo/Black</material>
     </gazebo>
-    <gazebo reference="front_right_tire_link">
+    <gazebo reference="front_right_wheel_link">
         <material>Gazebo/Black</material>
     </gazebo>
-    <gazebo reference="back_left_tire_link">
+    <gazebo reference="back_right_wheel_link">
         <material>Gazebo/Black</material>
     </gazebo>
-    <gazebo reference="back_right_tire_link">
+    <gazebo reference="back_left_wheel_link">
         <material>Gazebo/Black</material>
     </gazebo>
@@ -23,7 +23,4 @@
     </gazebo>
     <gazebo reference="camera_link">
-        <material>Gazebo/Black</material>
-    </gazebo>
-    <gazebo reference="imu_link">
         <material>Gazebo/Black</material>
     </gazebo>
@@ -46,5 +43,5 @@
           </plugin>
     </gazebo> -->
-    <gazebo>
+    <!-- <gazebo>
         <plugin name="gazebo_ros_planar_move" filename="libgazebo_ros_planar_move.so">
             <update_rate>100</update_rate>
@@ -52,15 +49,58 @@
             <publish_odom>true</publish_odom>
             <publish_odom_tf>true</publish_odom_tf>
-            <odometry_frame>odom_demo</odometry_frame>
-            <robot_base_frame>base_bottom_link</robot_base_frame>
+            <odometry_frame>odom</odometry_frame>
+            <robot_base_frame>chassis_base</robot_base_frame>
             <covariance_x>0.0001</covariance_x>
             <covariance_y>0.0001</covariance_y>
             <covariance_yaw>0.01</covariance_yaw>
           </plugin>
+    </gazebo> -->
+    <ros2_control name="GazeboSystem" type="system">
+        <hardware>
+            <plugin>gazebo_ros2_control/GazeboSystem</plugin>
+        </hardware>
+        <joint name="base_front_right_wheel_joint">
+            <command_interface name="velocity">
+                <param name="min">-10</param>
+                <param name="max">10</param>
+            </command_interface>
+            <state_interface name="position" />
+            <state_interface name="velocity" />
+        </joint>
+        <joint name="base_back_right_wheel_joint">
+            <command_interface name="velocity">
+                <param name="min">-10</param>
+                <param name="max">10</param>
+            </command_interface>
+            <state_interface name="position" />
+            <state_interface name="velocity" />
+        </joint>
+        <joint name="base_front_left_wheel_joint">
+            <command_interface name="velocity">
+                <param name="min">-10</param>
+                <param name="max">10</param>
+            </command_interface>
+            <state_interface name="position" />
+            <state_interface name="velocity" />
+        </joint>
+        <joint name="base_back_left_wheel_joint">
+            <command_interface name="velocity">
+                <param name="min">-10</param>
+                <param name="max">10</param>
+            </command_interface>
+            <state_interface name="position" />
+            <state_interface name="velocity" />
+        </joint>
+    </ros2_control>
+    <gazebo>
+        <plugin name="gazebo_ros2_control" filename="libgazebo_ros2_control.so">
+            <robot_sim_type>gazebo_ros2_control/GazeboSystem</robot_sim_type>
+            <parameters>$(find amr_description)/config/amr_controller.yaml</parameters>
+        </plugin>
     </gazebo>
     <gazebo reference="laser_scan">
         <sensor name="laser" type="ray">
             <pose> 0 0 0 0 0 0 </pose>
-            <visualize>false</visualize>
+            <visualize>true</visualize>
             <update_rate>10</update_rate>
             <ray>
@@ -105,17 +145,8 @@
             <plugin name="camera_controller" filename="libgazebo_ros_camera.so">
                 <frame_name>camera_link_optical</frame_name>
-                <!-- <imageTopicName>image_raw</imageTopicName>
-                <cameraInfoTopicName>camera_info</cameraInfoTopicName> -->
+                <imageTopicName>image_raw</imageTopicName>
+                <cameraInfoTopicName>camera_info</cameraInfoTopicName>
             </plugin>
         </sensor>
     </gazebo>
-    <gazebo reference="imu_link">
-        <sensor name="my_imu" type="imu">
-            <!-- ensure the sensor is active (required) -->
-            <always_on>true</always_on>
-            <update_rate>30</update_rate>
-            <plugin name="my_imu_plugin" filename="libgazebo_ros_imu_sensor.so">
-            </plugin>
-          </sensor>
-    </gazebo>
 </robot>

File: amr_description/urdf/amr_lidar.urdf.xacro (robot description, xacro)
@@ -1,10 +1,12 @@
 <?xml version="1.0"?>
 <robot xmlns:xacro="http://www.ros.org/wiki/xacro">
+    <xacro:property name="lidar_radius" value="0.03"/>
+    <xacro:property name="lidar_length" value="0.03"/>
     <link name="laser_scan">
         <visual>
             <geometry>
-                <cylinder radius="0.07" length="0.05"/>
+                <cylinder radius="${lidar_radius}" length="${lidar_length}"/>
             </geometry>
-            <origin xyz="0.0 0.0 0.0" rpy="0.0 0.0 0.0"/>
+            <origin xyz="0.0 ${lidar_radius} ${lidar_length/2}" rpy="0.0 0.0 0.0"/>
             <material name="black">
                 <color rgba="0.0 0.0 0.0 1.0"/>
@@ -13,5 +15,5 @@
         <collision>
             <geometry>
-                <cylinder radius="0.07" length="0.05"/>
+                <cylinder radius="${lidar_radius}" length="${lidar_length}"/>
             </geometry>
             <origin xyz="0.0 0.0 0.0" rpy="0.0 0.0 0.0"/>
@@ -21,6 +23,6 @@
     </link>
     <joint name="base_top_laser_scan_joint" type="fixed">
-        <origin xyz="-0.125 0.0 0.045" rpy="0.0 0.0 0.0"/>
-        <parent link="base_top_link"/>
+        <origin xyz="0.0 ${-chassis_width/2} 0.0" rpy="0.0 0.0 0.0"/>
+        <parent link="chassis_top"/>
         <child link="laser_scan"/>
     </joint>

File: amr_description/urdf/amrbase.urdf.xacro (robot description, xacro)
@@ -1,8 +1,13 @@
 <?xml version="1.0"?>
 <robot xmlns:xacro="http://www.ros.org/wiki/xacro">
+    <xacro:property name="chassis_length" value="0.5"/>
+    <xacro:property name="chassis_width" value="0.3"/>
+    <xacro:property name="chassis_height" value="0.0025"/>
+    <xacro:property name="wheel_radius" value="0.045"/>
+    <xacro:property name="wheel_length" value="0.04"/>
     <link name="base_bottom_link">
         <visual>
             <geometry>
-                <box size="0.5 0.25 0.02"/>
+                <box size="${chassis_length} ${chassis_width} ${chassis_height}"/>
             </geometry>
             <origin xyz="0.0 0.0 0.01" rpy="0.0 0.0 0.0"/>

File: amr_description/urdf/main.urdf.xacro (robot description, xacro)
@@ -2,8 +2,8 @@
 <robot xmlns:xacro="http://www.ros.org/wiki/xacro" name="amr">
     <xacro:include filename="inertial.urdf.xacro"/>
-    <xacro:include filename="amrbase.urdf.xacro"/>
+    <xacro:include filename="amr_core.urdf.xacro"/>
     <xacro:include filename="amr_lidar.urdf.xacro"/>
     <xacro:include filename="amr_camera.urdf.xacro"/>
-    <xacro:include filename="amr_imu.urdf.xacro"/>
+    <!-- <xacro:include filename="amr_imu.urdf.xacro"/> -->
     <xacro:include filename="amr_gazebo.urdf.xacro"/>
 </robot>
